File: hardware/braillekeyboard.kicad_sch (KiCad schematic)
At the start: 10 parts, among them U1 74HCT237, U2 ESP32-C3-WROOM-02

Commit message: Schematic inclusion
Parts:
- removed L0, L1, L2, L3, L4, L5, L6, L7: L, symbol Device:L
- removed U1: 74HCT237, symbol 74xx:74HCT237
- removed U2: ESP32-C3-WROOM-02, RF_Module:ESP32-C3-WROOM-02, symbol RF_Module:ESP32-C3-WROOM-02
- added C1: 100uF, symbol Device:C_Polarized
- added C2: 100nF, symbol Device:C
- added D1: 1N4007, Diode_THT:D_DO-41_SOD81_P10.16mm_Horizontal, symbol Diode:1N4007
- added J1, J2: Conn_01x15_Socket, symbol Connector:Conn_01x15_Socket
- added M1: Motor_DC, symbol Motor:Motor_DC
- added Q1: IRLZ44N, Package_TO_SOT_THT:TO-220-3_Vertical, symbol Transistor_FET:IRLZ44N
- added R1: 100, symbol Device:R
Connections:
- net GND: now also C1.2, C2.2, D1.2 (A), M1.2 (-), Q1.3 (S)
- new net: Q1.1 (G), R1.2
- new net +7.4V: C1.1, C2.1, D1.1 (K), M1.1 (+), Q1.2 (D)
- new net MOTOR_1: R1.1

Commit message: Atualizações de interface e hardware
Parts:
- added C10, C12, C4, C6, C8: 100nF, symbol Device:C
- added C11, C3, C5, C7, C9: 470uF, symbol Device:C_Polarized
- added D2, D3, D4, D5, D6: 1N4007, Diode_THT:D_DO-41_SOD81_P10.16mm_Horizontal, symbol Diode:1N4007
- added M2, M3, M4, M5, M6: Motor_DC, symbol Motor:Motor_DC
- added Q2, Q3, Q4, Q5, Q6: IRLZ44N, Package_TO_SOT_THT:TO-220-3_Vertical, symbol Transistor_FET:IRLZ44N
- added R11, R3, R5, R7, R9: 0, symbol Device:R
- added U1: LM2596, symbol Generic:Module_LM2596
- C1: value 100uF -> 470uF
- R1: value 100 -> 0
Connections:
- net GND: now also J1.14 (Pin_14), J2.2 (Pin_2), C10.2, C11.2, C12.2, C3.2, C4.2, C5.2, C6.2, C7.2, C8.2, C9.2, D2.2 (A), D3.2 (A), D4.2 (A), D5.2 (A), D6.2 (A), M2.2 (-), M3.2 (-), M4.2 (-), M5.2 (-), M6.2 (-), Q2.3 (S), Q3.3 (S), Q4.3 (S), Q5.3 (S), Q6.3 (S), U1.2 (GND_IN), U1.4 (GND_OUT)
- net VDD3_3: now reaches J2.1 (Pin_1)
- net D19: now reaches J2.10 (Pin_10)
- net D21: now reaches J2.11 (Pin_11)
- net RX0: now reaches J2.12 (Pin_12)
- net TX0: now reaches J2.13 (Pin_13)
- net D22: now reaches J2.14 (Pin_14)
- net D23: now reaches J2.15 (Pin_15)
- net D15: now reaches J2.3 (Pin_3)
- net D2: now reaches J2.4 (Pin_4)
- net D4: now reaches J2.5 (Pin_5)
- net D16: now reaches J2.6 (Pin_6)
- net D17: now reaches J2.7 (Pin_7)
- net D5: now reaches J2.8 (Pin_8)
- net D18: now reaches J2.9 (Pin_9)
- net EN: now reaches J1.1 (Pin_1)
- net D27: now reaches J1.10 (Pin_10)
- net D14: now reaches J1.11 (Pin_11)
- net D12: now reaches J1.12 (Pin_12)
- net D13: now reaches J1.13 (Pin_13)
- net VIN: now reaches J1.15 (Pin_15)
- net VP: now reaches J1.2 (Pin_2)
- net VN: now reaches J1.3 (Pin_3)
- net D34: now reaches J1.4 (Pin_4)
- net D35: now reaches J1.5 (Pin_5)
- net D32: now reaches J1.6 (Pin_6)
- net D33: now reaches J1.7 (Pin_7)
- net D25: now reaches J1.8 (Pin_8)
- net D26: now reaches J1.9 (Pin_9)
- net +7.4V renamed +7.5V
- net +7.5V: now also C10.1, C11.1, C12.1, C3.1, C4.1, C5.1, C6.1, C7.1, C8.1, C9.1, D2.1 (K), D3.1 (K), D4.1 (K), D5.1 (K), D6.1 (K), M2.1 (+), M3.1 (+), M4.1 (+), M5.1 (+), M6.1 (+), Q2.2 (D), Q3.2 (D), Q4.2 (D), Q5.2 (D), Q6.2 (D), U1.3 (VOUT)
- net MOTOR_1 renamed EN_MOTOR_1
- new net: Q3.1 (G), R5.2
- new net: Q6.1 (G), R11.2
- new net: Q5.1 (G), R9.2
- new net: Q4.1 (G), R7.2
- new net: Q2.1 (G), R3.2
- new net +12V: U1.1 (VIN)
Other:
- moved on the sheet: C1, C2, D1, J1, J2, M1, Q1, R1

Commit message: Atualização dos footprints
Parts:
- removed Q1, Q2, Q3, Q4, Q5, Q6: IRLZ44N, Package_TO_SOT_THT:TO-220-3_Vertical, symbol Transistor_FET:IRLZ44N
- added Q1, Q2, Q3, Q4, Q5, Q6: BC337, bc337:BC33716TA, symbol Transistor_BJT:BC337
- C1, C11, C3, C5, C7, C9: footprint (none) -> Capacitor_THT:CP_Radial_D12.5mm_P5.00mm
- C10, C12, C2, C4, C6, C8: footprint (none) -> Capacitor_THT:CP_Radial_D10.0mm_P7.50mm
- J1, J2: footprint (none) -> Connector_PinSocket_2.54mm:PinSocket_1x15_P2.54mm_Vertical
- R1, R11, R3, R5, R7, R9: footprint (none) -> Resistor_THT:R_Axial_DIN0617_L17.0mm_D6.0mm_P25.40mm_Horizontal
- U1: footprint (none) -> lm2596:LM2596_Module
Connections:
- net EN_MOTOR_1 is gone; now on net D21: R1.1
- net +7.5V: now also Q1.1 (C), Q2.1 (C), Q3.1 (C), Q4.1 (C), Q5.1 (C), Q6.1 (C)
- net D16: now also R11.1
- net D17: now also R7.1
- net D18: now also R9.1
- net D19: now also R3.1
- net D5: now also R5.1
- net GND: now also Q1.3 (E), Q2.3 (E), Q3.3 (E), Q4.3 (E), Q5.3 (E), Q6.3 (E)
- net at R5.2: now also Q2.2 (B)
- net at R11.2: now also Q6.2 (B)
- net at R1.2: now also Q1.2 (B)
- net at R9.2: now also Q5.2 (B)
- net at R7.2: now also Q3.2 (B)
- net at R3.2: now also Q4.2 (B)

Commit message: Reorganização dos componentes
Parts:
- added J3: Barrel_Jack_Switch, barreljack:BarrelJack_Horizontal, symbol Connector:Barrel_Jack_Switch
- C10, C12, C2, C4, C6, C8: footprint Capacitor_THT:CP_Radial_D10.0mm_P7.50mm -> Capacitor_THT:CP_Radial_D5.0mm_P2.50mm
Connections:
- net +12V: now also J3.1
- net GND: now also J3.2, J3.3
Changed lines of the file:
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@@
 	)
 	(junction
+		(at 35.56 119.38)
+		(diameter 0)
+		(color 0 0 0 0)
+	)
+	(junction
 		(at 181.61 115.57)
 		(diameter 0)
@@
 	)
 	(junction
+		(at 33.02 114.3)
+		(diameter 0)
+		(color 0 0 0 0)
+	)
+	(junction
 		(at 38.1 114.3)
 		(diameter 0)
@@
 	(wire
 		(pts
+			(xy 30.48 114.3) (xy 33.02 114.3)
+		)
+		(stroke
+			(width 0)
+			(type default)
+		)
+	)
+	(wire
+		(pts
 			(xy 120.65 58.42) (xy 120.65 60.96)
 		)
@@
 	(wire
 		(pts
+			(xy 30.48 119.38) (xy 35.56 119.38)
+		)
+		(stroke
+			(width 0)
+			(type default)
+		)
+	)
+	(wire
+		(pts
 			(xy 135.89 76.2) (xy 135.89 77.47)
 		)
@@
 	(wire
 		(pts
+			(xy 35.56 116.84) (xy 35.56 119.38)
+		)
+		(stroke
+			(width 0)
+			(type default)
+		)
+	)
+	(wire
+		(pts
 			(xy 260.35 58.42) (xy 260.35 60.96)
 		)
@@
 	(wire
 		(pts
+			(xy 30.48 116.84) (xy 35.56 116.84)
+		)
+		(stroke
+			(width 0)
+			(type default)
+		)
+	)
+	(wire
+		(pts
 			(xy 161.29 123.19) (xy 163.83 123.19)
 		)
@@
 	)
 	(symbol
+		(lib_id "Connector:Barrel_Jack_Switch")
+		(at 22.86 116.84 0)
+		(unit 1)
+		(exclude_from_sim no)
+		(in_bom yes)
+		(on_board yes)
+		(dnp no)
+		(fields_autoplaced yes)
+		(property "Reference" "J3"
+			(at 22.86 107.95 0)
+			(effects
+				(font
+					(size 1.27 1.27)
+				)
+			)
+		)
+		(property "Value" "Barrel_Jack_Switch"
+			(at 22.86 110.49 0)
+			(effects
+				(font
+					(size 1.27 1.27)
+				)
+			)
+		)
+		(property "Footprint" "barreljack:BarrelJack_Horizontal"
+			(at 24.13 117.856 0)
+			(effects
+				(font
+					(size 1.27 1.27)
+				)
+				(hide yes)
+			)
+		)
+		(property "Datasheet" "~"
+			(at 24.13 117.856 0)
+			(effects
+				(font
+					(size 1.27 1.27)
+				)
+				(hide yes)
+			)
+		)
+		(property "Description" "DC Barrel Jack with an internal switch"
+			(at 22.86 116.84 0)
+			(effects
+				(font
+					(size 1.27 1.27)
+				)
+				(hide yes)
+			)
+		)
+		(pin "3"
+		)
+		(pin "2"
+		)
+		(pin "1"
+		)
+		(instances
+			(project ""
+				(path "/18b850cf-544c-49d6-a580-a3bea7934356"
+					(reference "J3")
+					(unit 1)
+				)
+			)
+		)
+	)
+	(symbol
 		(lib_id "Device:R")
 		(at 106.68 123.19 90)
@@
 			)
 		)
-		(property "Footprint" "Capacitor_THT:CP_Radial_D10.0mm_P7.50mm"
+		(property "Footprint" "Capacitor_THT:CP_Radial_D5.0mm_P2.50mm"
 			(at 191.77 53.6448 0)
 			(effects
@@
 			)
 		)
-		(property "Footprint" "Capacitor_THT:CP_Radial_D10.0mm_P7.50mm"
+		(property "Footprint" "Capacitor_THT:CP_Radial_D5.0mm_P2.50mm"
 			(at 130.81 110.7948 0)
 			(effects
@@
 			)
 		)
-		(property "Footprint" "Capacitor_THT:CP_Radial_D10.0mm_P7.50mm"
+		(property "Footprint" "Capacitor_THT:CP_Radial_D5.0mm_P2.50mm"
 			(at 254 110.7948 0)
 			(effects
@@
 			)
 		)
-		(property "Footprint" "Capacitor_THT:CP_Radial_D10.0mm_P7.50mm"
+		(property "Footprint" "Capacitor_THT:CP_Radial_D5.0mm_P2.50mm"
 			(at 191.77 110.7948 0)
 			(effects
@@
 			)
 		)
-		(property "Footprint" "Capacitor_THT:CP_Radial_D10.0mm_P7.50mm"
+		(property "Footprint" "Capacitor_THT:CP_Radial_D5.0mm_P2.50mm"
 			(at 130.81 53.6448 0)
 			(effects
@@
 			)
 		)
-		(property "Footprint" "Capacitor_THT:CP_Radial_D10.0mm_P7.50mm"
+		(property "Footprint" "Capacitor_THT:CP_Radial_D5.0mm_P2.50mm"
 			(at 251.46 53.6448 0)
 			(effects

Commit message: PCB layout v1
Parts:
- M1, M4, M5, M6: footprint (none) -> Connector_JST:JST_XH_B2B-XH-AM_1x02_P2.50mm_Vertical
- M2: renamed from M3; footprint (none) -> Connector_JST:JST_XH_B2B-XH-AM_1x02_P2.50mm_Vertical
- M3: renamed from M2; footprint (none) -> Connector_JST:JST_XH_B2B-XH-AM_1x02_P2.50mm_Vertical
- renumbered C5 to C3, C6 to C4, C3 to C5, C4 to C6, D3 to D2, D2 to D3, Q4 to Q3, Q3 to Q4, R5 to R2, R7 to R4, R9 to R5, R11 to R6
Connections:
- net D17: now also R5.1; no longer R4.1
- net D18: now also R3.1; no longer R5.1
- net D19: now also R2.1; no longer R3.1
- net D5: now also R4.1; no longer R2.1
Changed lines of the file:
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@@
 		)
 	)
-	(global_label "D18"
+	(global_label "D17"
 		(shape bidirectional)
 		(at 220.98 66.04 180)
@@
 		)
 	)
-	(global_label "D19"
+	(global_label "D18"
 		(shape bidirectional)
 		(at 161.29 66.04 180)
@@
 		)
 	)
-	(global_label "D5"
+	(global_label "D19"
 		(shape bidirectional)
 		(at 100.33 123.19 180)
@@
 		)
 		(property "Intersheetrefs" "${INTERSHEET_REFS}"
-			(at 93.754 123.19 0)
+			(at 92.5445 123.19 0)
 			(effects
 				(font
@@
 		)
 	)
-	(global_label "D17"
+	(global_label "D5"
 		(shape bidirectional)
 		(at 161.29 123.19 180)
@@
 		)
 		(property "Intersheetrefs" "${INTERSHEET_REFS}"
-			(at 153.5045 123.19 0)
+			(at 154.714 123.19 0)
 			(effects
 				(font
@@
 		(on_board yes)
 		(dnp no)
-		(property "Reference" "C3"
+		(property "Reference" "C5"
 			(at 187.198 43.434 90)
 			(effects
@@
 			(project "braillekeyboard"
 				(path "/18b850cf-544c-49d6-a580-a3bea7934356"
-					(reference "C3")
+					(reference "C5")
 					(unit 1)
 				)
@@
 		(dnp no)
 		(fields_autoplaced yes)
-		(property "Reference" "Q4"
+		(property "Reference" "Q3"
 			(at 184.15 64.7699 0)
 			(effects
@@
 			(project "braillekeyboard"
 				(path "/18b850cf-544c-49d6-a580-a3bea7934356"
-					(reference "Q4")
+					(reference "Q3")
 					(unit 1)
 				)
@@
 		(on_board yes)
 		(dnp no)
-		(property "Reference" "D3"
+		(property "Reference" "D2"
 			(at 127.508 125.222 90)
 			(effects
@@
 			(project "braillekeyboard"
 				(path "/18b850cf-544c-49d6-a580-a3bea7934356"
-					(reference "D3")
+					(reference "D2")
 					(unit 1)
 				)
@@
 		(dnp no)
 		(fields_autoplaced yes)
-		(property "Reference" "R5"
+		(property "Reference" "R2"
 			(at 106.68 116.84 90)
 			(effects
@@
 			(project "braillekeyboard"
 				(path "/18b850cf-544c-49d6-a580-a3bea7934356"
-					(reference "R5")
+					(reference "R2")
 					(unit 1)
 				)
@@
 			)
 		)
-		(property "Footprint" ""
+		(property "Footprint" "Connector_JST:JST_XH_B2B-XH-AM_1x02_P2.50mm_Vertical"
 			(at 260.35 68.326 0)
 			(effects
@@
 		(dnp no)
 		(fields_autoplaced yes)
-		(property "Reference" "R11"
+		(property "Reference" "R6"
 			(at 229.87 116.84 90)
 			(effects
@@
 			(project "braillekeyboard"
 				(path "/18b850cf-544c-49d6-a580-a3bea7934356"
-					(reference "R11")
+					(reference "R6")
 					(unit 1)
 				)
@@
 		(on_board yes)
 		(dnp no)
-		(property "Reference" "D2"
+		(property "Reference" "D3"
 			(at 188.468 68.072 90)
 			(effects
@@
 			(project "braillekeyboard"
 				(path "/18b850cf-544c-49d6-a580-a3bea7934356"
-					(reference "D2")
+					(reference "D3")
 					(unit 1)
 				)
@@
 		(on_board yes)
 		(dnp no)
-		(property "Reference" "C5"
+		(property "Reference" "C3"
 			(at 126.238 100.584 90)
 			(effects
@@
 			(project "braillekeyboard"
 				(path "/18b850cf-544c-49d6-a580-a3bea7934356"
-					(reference "C5")
+					(reference "C3")
 					(unit 1)
 				)
@@
 		(on_board yes)
 		(dnp no)
-		(property "Reference" "M3"
+		(property "Reference" "M2"
 			(at 143.256 124.714 0)
 			(effects
@@
 			)
 		)
-		(property "Footprint" ""
+		(property "Footprint" "Connector_JST:JST_XH_B2B-XH-AM_1x02_P2.50mm_Vertical"
 			(at 139.7 125.476 0)
 			(effects
@@
 			(project "braillekeyboard"
 				(path "/18b850cf-544c-49d6-a580-a3bea7934356"
-					(reference "M3")
+					(reference "M2")
 					(unit 1)
 				)
@@
 		(on_board yes)
 		(dnp no)
-		(property "Reference" "C4"
+		(property "Reference" "C6"
 			(at 191.008 50.8 90)
 			(effects
@@
 			(project "braillekeyboard"
 				(path "/18b850cf-544c-49d6-a580-a3bea7934356"
-					(reference "C4")
+					(reference "C6")
 					(unit 1)
 				)
@@
 		(dnp no)
 		(fields_autoplaced yes)
-		(property "Reference" "R9"
+		(property "Reference" "R5"
 			(at 227.33 59.69 90)
 			(effects
@@
 			(project "braillekeyboard"
 				(path "/18b850cf-544c-49d6-a580-a3bea7934356"
-					(reference "R9")
+					(reference "R5")
 					(unit 1)
 				)
@@
 		(on_board yes)
 		(dnp no)
-		(property "Reference" "C6"
+		(property "Reference" "C4"
 			(at 130.048 107.95 90)
 			(effects
@@
 			(project "braillekeyboard"
 				(path "/18b850cf-544c-49d6-a580-a3bea7934356"
-					(reference "C6")
+					(reference "C4")
 					(unit 1)
 				)
@@
 		(on_board yes)
 		(dnp no)
-		(property "Reference" "M2"
+		(property "Reference" "M3"
 			(at 204.216 67.564 0)
 			(effects
@@
 			)
 		)
-		(property "Footprint" ""
+		(property "Footprint" "Connector_JST:JST_XH_B2B-XH-AM_1x02_P2.50mm_Vertical"
 			(at 200.66 68.326 0)
 			(effects
@@
 			(project "braillekeyboard"
 				(path "/18b850cf-544c-49d6-a580-a3bea7934356"
-					(reference "M2")
+					(reference "M3")
 					(unit 1)
 				)
@@
 			)
 		)
-		(property "Footprint" ""
+		(property "Footprint" "Connector_JST:JST_XH_B2B-XH-AM_1x02_P2.50mm_Vertical"
 			(at 200.66 125.476 0)
 			(effects
@@
 			)
 		)
-		(property "Footprint" ""
+		(property "Footprint" "Connector_JST:JST_XH_B2B-XH-AM_1x02_P2.50mm_Vertical"
 			(at 139.7 68.326 0)
 			(effects
@@
 			)
 		)
-		(property "Footprint" ""
+		(property "Footprint" "Connector_JST:JST_XH_B2B-XH-AM_1x02_P2.50mm_Vertical"
 			(at 262.89 125.476 0)
 			(effects
@@
 		(dnp no)
 		(fields_autoplaced yes)
-		(property "Reference" "R7"
+		(property "Reference" "R4"
 			(at 167.64 116.84 90)
 			(effects
@@
 			(project "braillekeyboard"
 				(path "/18b850cf-544c-49d6-a580-a3bea7934356"
-					(reference "R7")
+					(reference "R4")
 					(unit 1)
 				)
@@
 		(dnp no)
 		(fields_autoplaced yes)
-		(property "Reference" "Q3"
+		(property "Reference" "Q4"
 			(at 184.15 121.9199 0)
 			(effects
@@
 			(project "braillekeyboard"
 				(path "/18b850cf-544c-49d6-a580-a3bea7934356"
-					(reference "Q3")
+					(reference "Q4")
 					(unit 1)
 				)
