File: hardware/hardware_V0/braillekeyboard.kicad_sch (KiCad schematic)
At the start: 40 parts, among them J1 Conn_01x15_Socket, J2 Conn_01x15_Socket, J3 Barrel_Jack_Switch, M1 Motor_DC, M2 Motor_DC, M3 Motor_DC, M4 Motor_DC, M5 Motor_DC, M6 Motor_DC, Q1 BC337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

Commit message: Subdivisão do hardware para implementação da nova versão
Parts:
- added C13: 0.33uF, 330u:CAPPRD350W60D825H1300, symbol Device:C
- added C14: 0.1uF, 100u:615R100GAD10, symbol Device:C
- added U2: LM7805_TO220, Package_TO_SOT_THT:TO-220-3_Vertical, symbol Regulator_Linear:LM7805_TO220
- C1, C11, C3, C5, C7, C9: footprint Capacitor_THT:CP_Radial_D12.5mm_P5.00mm -> 470u:CAPPRD500W60D1050H1750
- C10, C12, C2, C4, C6, C8: footprint Capacitor_THT:CP_Radial_D5.0mm_P2.50mm -> 100u:615R100GAD10
Connections:
- net +12V: now also C13.1, U2.1 (VI)
- net GND: now also C13.2, C14.2, U2.2 (GND)
- net VIN renamed VDD5
- net VDD5: now also C14.1, U2.3 (VO)
Other:
- moved on the sheet: J3, U1
