File: hardware/hardware_V1/braillekeyboard.kicad_pcb (KiCad board)
At the start: 2 copper layers, 43 parts, among them J1 Conn_01x15_Socket, J2 Conn_01x15_Socket, J3 Barrel_Jack_Switch, M1 Motor_DC, M2 Motor_DC, M3 Motor_DC, M4 Motor_DC, M5 Motor_DC, M6 Motor_DC, Q1 BC337, Q2 BC337, Q3 BC337, Q4 BC337, Q5 BC337, Q6 BC337, U1 LM2596, U2 LM7805_TO220

Commit message: Inclusão do latch no circuito, ampliação para 36 motores
Parts:
- added C15: 470uF, 470u:CAPPRD500W60D1050H1750, F.Cu at (110.7, 262.9)
- added C16: 100nF, 100u:615R100GAD10, F.Cu at (53.6, 274.5)
- added C17: 470uF, 470u:CAPPRD500W60D1050H1750, F.Cu at (110.7, 274.6)
- added C18: 100nF, 100u:615R100GAD10, F.Cu at (64.8, 274.5)
- added C19: 470uF, 470u:CAPPRD500W60D1050H1750, F.Cu at (110.7, 286.3)
- added C20: 100nF, 100u:615R100GAD10, F.Cu at (76.0, 274.5)
- added C21: 470uF, 470u:CAPPRD500W60D1050H1750, F.Cu at (110.7, 298.0)
- added C22: 100nF, 100u:615R100GAD10, F.Cu at (87.2, 274.5)
- added C23: 470uF, 470u:CAPPRD500W60D1050H1750, F.Cu at (110.7, 309.7)
- added C24: 100nF, 100u:615R100GAD10, F.Cu at (-13.6, 296.7)
- added C25: 470uF, 470u:CAPPRD500W60D1050H1750, F.Cu at (110.7, 321.4)
- added C26: 100nF, 100u:615R100GAD10, F.Cu at (-2.37, 296.7)
- added C27: 470uF, 470u:CAPPRD500W60D1050H1750, F.Cu at (122.4, 262.9)
- added C28: 100nF, 100u:615R100GAD10, F.Cu at (8.83, 296.7)
- added C29: 470uF, 470u:CAPPRD500W60D1050H1750, F.Cu at (122.4, 274.6)
- added C30: 100nF, 100u:615R100GAD10, F.Cu at (20.0, 296.7)
- added C31: 470uF, 470u:CAPPRD500W60D1050H1750, F.Cu at (122.4, 286.3)
- added C32: 100nF, 100u:615R100GAD10, F.Cu at (31.2, 296.7)
- added C33: 470uF, 470u:CAPPRD500W60D1050H1750, F.Cu at (122.4, 298.0)
- added C34: 100nF, 100u:615R100GAD10, F.Cu at (42.4, 296.7)
- added C35: 470uF, 470u:CAPPRD500W60D1050H1750, F.Cu at (122.4, 309.7)
- added C36: 100nF, 100u:615R100GAD10, F.Cu at (53.6, 296.7)
- added C37: 470uF, 470u:CAPPRD500W60D1050H1750, F.Cu at (122.4, 321.4)
- added C38: 100nF, 100u:615R100GAD10, F.Cu at (64.8, 296.7)
- added C39: 470uF, 470u:CAPPRD500W60D1050H1750, F.Cu at (134.1, 262.9)
- added C40: 100nF, 100u:615R100GAD10, F.Cu at (76.0, 296.7)
- added C41: 470uF, 470u:CAPPRD500W60D1050H1750, F.Cu at (134.1, 274.6)
- added C42: 100nF, 100u:615R100GAD10, F.Cu at (87.2, 296.7)
- added C43: 470uF, 470u:CAPPRD500W60D1050H1750, F.Cu at (134.1, 286.3)
- added C44: 100nF, 100u:615R100GAD10, F.Cu at (-13.6, 318.9)
- added C45: 470uF, 470u:CAPPRD500W60D1050H1750, F.Cu at (134.1, 298.0)
- added C46: 100nF, 100u:615R100GAD10, F.Cu at (-2.37, 318.9)
- added C47: 470uF, 470u:CAPPRD500W60D1050H1750, F.Cu at (134.1, 309.7)
- added C48: 100nF, 100u:615R100GAD10, F.Cu at (8.83, 318.9)
- added C49: 470uF, 470u:CAPPRD500W60D1050H1750, F.Cu at (134.1, 321.4)
- added C50: 100nF, 100u:615R100GAD10, F.Cu at (20.0, 318.9)
- added C51: 470uF, 470u:CAPPRD500W60D1050H1750, F.Cu at (145.8, 262.9)
- added C52: 100nF, 100u:615R100GAD10, F.Cu at (31.2, 318.9)
- added C53: 470uF, 470u:CAPPRD500W60D1050H1750, F.Cu at (145.8, 274.6)
- added C54: 100nF, 100u:615R100GAD10, F.Cu at (42.4, 318.9)
- added C55: 470uF, 470u:CAPPRD500W60D1050H1750, F.Cu at (145.8, 286.3)
- added C56: 100nF, 100u:615R100GAD10, F.Cu at (53.6, 318.9)
- added C57: 470uF, 470u:CAPPRD500W60D1050H1750, F.Cu at (145.8, 298.0)
- added C58: 100nF, 100u:615R100GAD10, F.Cu at (64.8, 318.9)
- added C59: 470uF, 470u:CAPPRD500W60D1050H1750, F.Cu at (145.8, 309.7)
- added C60: 100nF, 100u:615R100GAD10, F.Cu at (76.0, 318.9)
- added C61: 470uF, 470u:CAPPRD500W60D1050H1750, F.Cu at (145.8, 321.4)
- added C62: 100nF, 100u:615R100GAD10, F.Cu at (87.2, 318.9)
- added C63: 470uF, 470u:CAPPRD500W60D1050H1750, F.Cu at (157.5, 262.9)
- added C64: 100nF, 100u:615R100GAD10, F.Cu at (-13.6, 341.1)
- added C65: 470uF, 470u:CAPPRD500W60D1050H1750, F.Cu at (157.5, 274.6)
- added C66: 100nF, 100u:615R100GAD10, F.Cu at (-2.37, 341.1)
- added C67: 470uF, 470u:CAPPRD500W60D1050H1750, F.Cu at (157.5, 286.3)
- added C68: 100nF, 100u:615R100GAD10, F.Cu at (8.83, 341.1)
- added C69: 470uF, 470u:CAPPRD500W60D1050H1750, F.Cu at (157.5, 298.0)
- added C70: 100nF, 100u:615R100GAD10, F.Cu at (20.0, 341.1)
- added C71: 470uF, 470u:CAPPRD500W60D1050H1750, F.Cu at (157.5, 309.7)
- added C72: 100nF, 100u:615R100GAD10, F.Cu at (31.2, 341.1)
- added C73: 470uF, 470u:CAPPRD500W60D1050H1750, F.Cu at (157.5, 321.4)
- added C74: 100nF, 100u:615R100GAD10, F.Cu at (42.4, 341.1)
- added D10: 1N4007, Diode_THT:D_DO-41_SOD81_P10.16mm_Horizontal, F.Cu at (112.1, 199.3)
- added D11: 1N4007, Diode_THT:D_DO-41_SOD81_P10.16mm_Horizontal, F.Cu at (112.1, 203.5)
- added D12: 1N4007, Diode_THT:D_DO-41_SOD81_P10.16mm_Horizontal, F.Cu at (112.1, 207.8)
- added D13: 1N4007, Diode_THT:D_DO-41_SOD81_P10.16mm_Horizontal, F.Cu at (126.0, 161.0)
- added D14: 1N4007, Diode_THT:D_DO-41_SOD81_P10.16mm_Horizontal, F.Cu at (126.0, 165.3)
- added D15: 1N4007, Diode_THT:D_DO-41_SOD81_P10.16mm_Horizontal, F.Cu at (126.0, 169.5)
- added D16: 1N4007, Diode_THT:D_DO-41_SOD81_P10.16mm_Horizontal, F.Cu at (126.0, 173.8)
- added D17: 1N4007, Diode_THT:D_DO-41_SOD81_P10.16mm_Horizontal, F.Cu at (126.0, 178.0)
- added D18: 1N4007, Diode_THT:D_DO-41_SOD81_P10.16mm_Horizontal, F.Cu at (126.0, 182.3)
- added D19: 1N4007, Diode_THT:D_DO-41_SOD81_P10.16mm_Horizontal, F.Cu at (126.0, 186.5)
- added D20: 1N4007, Diode_THT:D_DO-41_SOD81_P10.16mm_Horizontal, F.Cu at (126.0, 190.8)
- added D21: 1N4007, Diode_THT:D_DO-41_SOD81_P10.16mm_Horizontal, F.Cu at (126.0, 195.0)
- added D22: 1N4007, Diode_THT:D_DO-41_SOD81_P10.16mm_Horizontal, F.Cu at (126.0, 199.3)
- added D23: 1N4007, Diode_THT:D_DO-41_SOD81_P10.16mm_Horizontal, F.Cu at (126.0, 203.5)
- added D24: 1N4007, Diode_THT:D_DO-41_SOD81_P10.16mm_Horizontal, F.Cu at (126.0, 207.8)
- added D25: 1N4007, Diode_THT:D_DO-41_SOD81_P10.16mm_Horizontal, F.Cu at (139.9, 161.0)
- added D26: 1N4007, Diode_THT:D_DO-41_SOD81_P10.16mm_Horizontal, F.Cu at (139.9, 165.3)
- added D27: 1N4007, Diode_THT:D_DO-41_SOD81_P10.16mm_Horizontal, F.Cu at (139.9, 169.5)
- added D28: 1N4007, Diode_THT:D_DO-41_SOD81_P10.16mm_Horizontal, F.Cu at (139.9, 173.8)
- added D29: 1N4007, Diode_THT:D_DO-41_SOD81_P10.16mm_Horizontal, F.Cu at (139.9, 178.0)
- added D30: 1N4007, Diode_THT:D_DO-41_SOD81_P10.16mm_Horizontal, F.Cu at (139.9, 182.3)
- added D31: 1N4007, Diode_THT:D_DO-41_SOD81_P10.16mm_Horizontal, F.Cu at (139.9, 186.5)
- added D32: 1N4007, Diode_THT:D_DO-41_SOD81_P10.16mm_Horizontal, F.Cu at (139.9, 190.8)
- added D33: 1N4007, Diode_THT:D_DO-41_SOD81_P10.16mm_Horizontal, F.Cu at (139.9, 195.0)
- added D34: 1N4007, Diode_THT:D_DO-41_SOD81_P10.16mm_Horizontal, F.Cu at (139.9, 199.3)
- added D35: 1N4007, Diode_THT:D_DO-41_SOD81_P10.16mm_Horizontal, F.Cu at (139.9, 203.5)
- added D36: 1N4007, Diode_THT:D_DO-41_SOD81_P10.16mm_Horizontal, F.Cu at (139.9, 207.8)
- added D7: 1N4007, Diode_THT:D_DO-41_SOD81_P10.16mm_Horizontal, F.Cu at (112.1, 186.5)
- added D8: 1N4007, Diode_THT:D_DO-41_SOD81_P10.16mm_Horizontal, F.Cu at (112.1, 190.8)
- added D9: 1N4007, Diode_THT:D_DO-41_SOD81_P10.16mm_Horizontal, F.Cu at (112.1, 195.0)
- added M10: Motor_DC, Connector_JST:JST_XH_B2B-XH-AM_1x02_P2.50mm_Vertical, F.Cu at (123.1, 236.7)
- added M11: Motor_DC, Connector_JST:JST_XH_B2B-XH-AM_1x02_P2.50mm_Vertical, F.Cu at (123.1, 244.5)
- added M12: Motor_DC, Connector_JST:JST_XH_B2B-XH-AM_1x02_P2.50mm_Vertical, F.Cu at (123.1, 252.3)
- added M13: Motor_DC, Connector_JST:JST_XH_B2B-XH-AM_1x02_P2.50mm_Vertical, F.Cu at (132.6, 213.3)
- added M14: Motor_DC, Connector_JST:JST_XH_B2B-XH-AM_1x02_P2.50mm_Vertical, F.Cu at (132.6, 221.1)
- added M15: Motor_DC, Connector_JST:JST_XH_B2B-XH-AM_1x02_P2.50mm_Vertical, F.Cu at (132.6, 228.9)
- added M16: Motor_DC, Connector_JST:JST_XH_B2B-XH-AM_1x02_P2.50mm_Vertical, F.Cu at (132.6, 236.7)
- added M17: Motor_DC, Connector_JST:JST_XH_B2B-XH-AM_1x02_P2.50mm_Vertical, F.Cu at (132.6, 244.5)
- added M18: Motor_DC, Connector_JST:JST_XH_B2B-XH-AM_1x02_P2.50mm_Vertical, F.Cu at (132.6, 252.3)
- added M19: Motor_DC, Connector_JST:JST_XH_B2B-XH-AM_1x02_P2.50mm_Vertical, F.Cu at (142.0, 213.3)
- added M20: Motor_DC, Connector_JST:JST_XH_B2B-XH-AM_1x02_P2.50mm_Vertical, F.Cu at (142.0, 221.1)
- added M21: Motor_DC, Connector_JST:JST_XH_B2B-XH-AM_1x02_P2.50mm_Vertical, F.Cu at (142.0, 228.9)
- added M22: Motor_DC, Connector_JST:JST_XH_B2B-XH-AM_1x02_P2.50mm_Vertical, F.Cu at (142.0, 236.7)
- added M23: Motor_DC, Connector_JST:JST_XH_B2B-XH-AM_1x02_P2.50mm_Vertical, F.Cu at (142.0, 244.5)
- added M24: Motor_DC, Connector_JST:JST_XH_B2B-XH-AM_1x02_P2.50mm_Vertical, F.Cu at (142.0, 252.3)
- added M25: Motor_DC, Connector_JST:JST_XH_B2B-XH-AM_1x02_P2.50mm_Vertical, F.Cu at (151.5, 213.3)
- added M26: Motor_DC, Connector_JST:JST_XH_B2B-XH-AM_1x02_P2.50mm_Vertical, F.Cu at (151.5, 221.1)
- added M27: Motor_DC, Connector_JST:JST_XH_B2B-XH-AM_1x02_P2.50mm_Vertical, F.Cu at (151.5, 228.9)
- added M28: Motor_DC, Connector_JST:JST_XH_B2B-XH-AM_1x02_P2.50mm_Vertical, F.Cu at (151.5, 236.7)
- added M29: Motor_DC, Connector_JST:JST_XH_B2B-XH-AM_1x02_P2.50mm_Vertical, F.Cu at (151.5, 244.5)
- added M30: Motor_DC, Connector_JST:JST_XH_B2B-XH-AM_1x02_P2.50mm_Vertical, F.Cu at (151.5, 252.3)
- added M31: Motor_DC, Connector_JST:JST_XH_B2B-XH-AM_1x02_P2.50mm_Vertical, F.Cu at (160.9, 213.3)
- added M32: Motor_DC, Connector_JST:JST_XH_B2B-XH-AM_1x02_P2.50mm_Vertical, F.Cu at (160.9, 221.1)
- added M33: Motor_DC, Connector_JST:JST_XH_B2B-XH-AM_1x02_P2.50mm_Vertical, F.Cu at (160.9, 228.9)
- added M34: Motor_DC, Connector_JST:JST_XH_B2B-XH-AM_1x02_P2.50mm_Vertical, F.Cu at (160.9, 236.7)
- added M35: Motor_DC, Connector_JST:JST_XH_B2B-XH-AM_1x02_P2.50mm_Vertical, F.Cu at (160.9, 244.5)
- added M36: Motor_DC, Connector_JST:JST_XH_B2B-XH-AM_1x02_P2.50mm_Vertical, F.Cu at (160.9, 252.3)
- added M7: Motor_DC, Connector_JST:JST_XH_B2B-XH-AM_1x02_P2.50mm_Vertical, F.Cu at (123.1, 213.3)
- added M8: Motor_DC, Connector_JST:JST_XH_B2B-XH-AM_1x02_P2.50mm_Vertical, F.Cu at (123.1, 221.1)
- added M9: Motor_DC, Connector_JST:JST_XH_B2B-XH-AM_1x02_P2.50mm_Vertical, F.Cu at (123.1, 228.9)
- added Q10: BC337, bc337:BC33716TA, F.Cu at (83.5, 162.7)
- added Q11: BC337, bc337:BC33716TA, F.Cu at (83.5, 169.5)
- added Q12: BC337, bc337:BC33716TA, F.Cu at (83.5, 176.3)
- added Q13: BC337, bc337:BC33716TA, F.Cu at (83.5, 183.1)
- added Q14: BC337, bc337:BC33716TA, F.Cu at (83.5, 189.8)
- added Q15: BC337, bc337:BC33716TA, F.Cu at (83.5, 196.6)
- added Q16: BC337, bc337:BC33716TA, F.Cu at (83.5, 203.4)
- added Q17: BC337, bc337:BC33716TA, F.Cu at (83.5, 210.2)
- added Q18: BC337, bc337:BC33716TA, F.Cu at (83.5, 216.9)
- added Q19: BC337, bc337:BC33716TA, F.Cu at (93.2, 162.7)
- added Q20: BC337, bc337:BC33716TA, F.Cu at (93.2, 169.5)
- added Q21: BC337, bc337:BC33716TA, F.Cu at (93.2, 176.3)
- added Q22: BC337, bc337:BC33716TA, F.Cu at (93.2, 183.1)
- added Q23: BC337, bc337:BC33716TA, F.Cu at (93.2, 189.8)
- added Q24: BC337, bc337:BC33716TA, F.Cu at (93.2, 196.6)
- added Q25: BC337, bc337:BC33716TA, F.Cu at (93.2, 203.4)
- added Q26: BC337, bc337:BC33716TA, F.Cu at (93.2, 210.2)
- added Q27: BC337, bc337:BC33716TA, F.Cu at (93.2, 216.9)
- added Q28: BC337, bc337:BC33716TA, F.Cu at (102.8, 162.7)
- added Q29: BC337, bc337:BC33716TA, F.Cu at (102.8, 169.5)
- added Q30: BC337, bc337:BC33716TA, F.Cu at (102.8, 176.3)
- added Q31: BC337, bc337:BC33716TA, F.Cu at (102.8, 183.1)
- added Q32: BC337, bc337:BC33716TA, F.Cu at (102.8, 189.8)
- added Q33: BC337, bc337:BC33716TA, F.Cu at (102.8, 196.6)
- added Q34: BC337, bc337:BC33716TA, F.Cu at (102.8, 203.4)
- added Q35: BC337, bc337:BC33716TA, F.Cu at (102.8, 210.2)
- added Q36: BC337, bc337:BC33716TA, F.Cu at (102.8, 216.9)
- added Q7: BC337, bc337:BC33716TA, F.Cu at (73.9, 203.4)
- added Q8: BC337, bc337:BC33716TA, F.Cu at (73.9, 210.2)
- added Q9: BC337, bc337:BC33716TA, F.Cu at (73.9, 216.9)
- added R10: 1k, Resistor_THT:R_Axial_DIN0617_L17.0mm_D6.0mm_P25.40mm_Horizontal, F.Cu at (170.9, 213.8)
- added R11: 0, Resistor_THT:R_Axial_DIN0617_L17.0mm_D6.0mm_P25.40mm_Horizontal, F.Cu at (-14.4, 208.0)
- added R12: 0, Resistor_THT:R_Axial_DIN0617_L17.0mm_D6.0mm_P25.40mm_Horizontal, F.Cu at (-14.4, 215.5)
- added R13: 0, Resistor_THT:R_Axial_DIN0617_L17.0mm_D6.0mm_P25.40mm_Horizontal, F.Cu at (-14.4, 223.1)
- added R14: 0, Resistor_THT:R_Axial_DIN0617_L17.0mm_D6.0mm_P25.40mm_Horizontal, F.Cu at (-14.4, 230.6)
- added R15: 0, Resistor_THT:R_Axial_DIN0617_L17.0mm_D6.0mm_P25.40mm_Horizontal, F.Cu at (-14.4, 238.2)
- added R16: 0, Resistor_THT:R_Axial_DIN0617_L17.0mm_D6.0mm_P25.40mm_Horizontal, F.Cu at (-14.4, 245.7)
- added R17: 0, Resistor_THT:R_Axial_DIN0617_L17.0mm_D6.0mm_P25.40mm_Horizontal, F.Cu at (-14.4, 253.3)
- added R18: 0, Resistor_THT:R_Axial_DIN0617_L17.0mm_D6.0mm_P25.40mm_Horizontal, F.Cu at (15.0, 162.7)
- added R19: 0, Resistor_THT:R_Axial_DIN0617_L17.0mm_D6.0mm_P25.40mm_Horizontal, F.Cu at (15.0, 170.2)
- added R20: 0, Resistor_THT:R_Axial_DIN0617_L17.0mm_D6.0mm_P25.40mm_Horizontal, F.Cu at (15.0, 177.8)
- added R21: 0, Resistor_THT:R_Axial_DIN0617_L17.0mm_D6.0mm_P25.40mm_Horizontal, F.Cu at (15.0, 185.3)
- added R22: 0, Resistor_THT:R_Axial_DIN0617_L17.0mm_D6.0mm_P25.40mm_Horizontal, F.Cu at (15.0, 192.9)
- added R23: 0, Resistor_THT:R_Axial_DIN0617_L17.0mm_D6.0mm_P25.40mm_Horizontal, F.Cu at (15.0, 200.4)
- added R24: 0, Resistor_THT:R_Axial_DIN0617_L17.0mm_D6.0mm_P25.40mm_Horizontal, F.Cu at (15.0, 208.0)
- added R25: 0, Resistor_THT:R_Axial_DIN0617_L17.0mm_D6.0mm_P25.40mm_Horizontal, F.Cu at (15.0, 215.5)
- added R26: 0, Resistor_THT:R_Axial_DIN0617_L17.0mm_D6.0mm_P25.40mm_Horizontal, F.Cu at (15.0, 223.1)
- added R27: 0, Resistor_THT:R_Axial_DIN0617_L17.0mm_D6.0mm_P25.40mm_Horizontal, F.Cu at (15.0, 230.6)
- added R28: 0, Resistor_THT:R_Axial_DIN0617_L17.0mm_D6.0mm_P25.40mm_Horizontal, F.Cu at (15.0, 238.2)
- added R29: 0, Resistor_THT:R_Axial_DIN0617_L17.0mm_D6.0mm_P25.40mm_Horizontal, F.Cu at (15.0, 245.7)
- added R30: 0, Resistor_THT:R_Axial_DIN0617_L17.0mm_D6.0mm_P25.40mm_Horizontal, F.Cu at (15.0, 253.3)
- added R31: 0, Resistor_THT:R_Axial_DIN0617_L17.0mm_D6.0mm_P25.40mm_Horizontal, F.Cu at (44.3, 162.7)
- added R32: 0, Resistor_THT:R_Axial_DIN0617_L17.0mm_D6.0mm_P25.40mm_Horizontal, F.Cu at (44.3, 170.2)
- added R33: 0, Resistor_THT:R_Axial_DIN0617_L17.0mm_D6.0mm_P25.40mm_Horizontal, F.Cu at (44.3, 177.8)
- added R34: 0, Resistor_THT:R_Axial_DIN0617_L17.0mm_D6.0mm_P25.40mm_Horizontal, F.Cu at (44.3, 185.3)
- added R35: 0, Resistor_THT:R_Axial_DIN0617_L17.0mm_D6.0mm_P25.40mm_Horizontal, F.Cu at (44.3, 192.9)
- added R36: 0, Resistor_THT:R_Axial_DIN0617_L17.0mm_D6.0mm_P25.40mm_Horizontal, F.Cu at (44.3, 200.4)
- added R37: 0, Resistor_THT:R_Axial_DIN0617_L17.0mm_D6.0mm_P25.40mm_Horizontal, F.Cu at (44.3, 208.0)
- added R38: 0, Resistor_THT:R_Axial_DIN0617_L17.0mm_D6.0mm_P25.40mm_Horizontal, F.Cu at (44.3, 215.5)
- added R39: 0, Resistor_THT:R_Axial_DIN0617_L17.0mm_D6.0mm_P25.40mm_Horizontal, F.Cu at (44.3, 223.1)
- added R40: 0, Resistor_THT:R_Axial_DIN0617_L17.0mm_D6.0mm_P25.40mm_Horizontal, F.Cu at (44.3, 230.6)
- added R7: 1k, Resistor_THT:R_Axial_DIN0617_L17.0mm_D6.0mm_P25.40mm_Horizontal, F.Cu at (170.9, 191.2)
- added R8: 1k, Resistor_THT:R_Axial_DIN0617_L17.0mm_D6.0mm_P25.40mm_Horizontal, F.Cu at (170.9, 198.7)
- added R9: 1k, Resistor_THT:R_Axial_DIN0617_L17.0mm_D6.0mm_P25.40mm_Horizontal, F.Cu at (170.9, 206.3)
- added U3: TPIC6595, tpic6595:DIP794W53P254L2540H508Q20N, F.Cu at (96.4, 64.4)
- added U4: TPIC6595, tpic6595:DIP794W53P254L2540H508Q20N, F.Cu at (96.4, 95.3)
- added U5: TPIC6595, tpic6595:DIP794W53P254L2540H508Q20N, F.Cu at (96.4, 126.1)
- added U6: TPIC6595, tpic6595:DIP794W53P254L2540H508Q20N, F.Cu at (207.2, 173.1)
- moved D1 334.1 mm to (560.5, 141.1)
- moved D2 333.5 mm to (560.5, 154.6)
- moved D3 333.1 mm to (560.5, 168.1)
- moved D4 332.6 mm to (560.5, 181.6)
- moved D5 332.0 mm to (560.5, 195.1)
- moved D6 331.5 mm to (560.5, 208.6)
- moved M1 330.0 mm to (564.5, 135.8)
- moved M2 329.5 mm to (564.5, 149.3)
- moved M3 329.3 mm to (564.5, 162.4)
- moved M4 328.5 mm to (564.5, 175.1)
- moved M5 328.0 mm to (564.5, 188.8)
- moved C2 327.9 mm to (554.3, 135.8)
- moved C1 327.8 mm to (530.1, 135.8)
- moved M6 327.7 mm to (564.5, 203.2)
- moved C4 327.4 mm to (554.3, 149.3)
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Connections:
- R1 pad 1: D21 -> CH1_MOTOR_1
- R2 pad 1: D19 -> CH1_MOTOR_2
- R3 pad 1: D18 -> CH1_MOTOR_3
- R4 pad 1: D5 -> CH1_MOTOR_4
- R5 pad 1: D17 -> CH1_MOTOR_5
- R6 pad 1: D16 -> CH1_MOTOR_6
Routing:
- net VCC7_5: track 0.00 -> 324.0 mm
- net D16: track 0.00 -> 44.8 mm
- net D17: track 0.00 -> 44.2 mm
- net D5: track 0.00 -> 25.3 mm
- net D18: track 0.00 -> 24.3 mm
- net D19: track 0.00 -> 24.3 mm
- net D21: track 0.00 -> 16.3 mm
- net Net-(Q3-B): track 0.00 -> 8.69 mm
- net Net-(Q4-B): track 0.00 -> 8.69 mm
- net Net-(Q2-B): track 0.00 -> 8.69 mm
- net Net-(Q1-B): track 0.00 -> 8.69 mm
- net Net-(Q6-B): track 0.00 -> 8.69 mm
- net Net-(Q5-B): track 0.00 -> 8.69 mm
